Commit message: controllerbelegung angepasst

File: src/lotti2_moveit_config/config/Lotti2.ros2_control.xacro (robot description, xacro)
@@ -56,12 +56,4 @@
                 <state_interface name="velocity"/>
             </joint>
-            <joint name="arm7_joint">
-                <command_interface name="position"/>
-                <command_interface name="velocity"/>
-                <state_interface name="position">
-                  <param name="initial_value">${initial_positions['arm7_joint']}</param>
-                </state_interface>
-                <state_interface name="velocity"/>
-            </joint>
         </ros2_control>
     </xacro:macro>
