Commit message: arm working

File: src/lotti2_control/description/ros2_control/Lotti2.ros2_control.xacro (robot description, xacro)
@@ -108,4 +108,10 @@
             <state_interface name="velocity"/>
         </joint>
+        <joint name="arm7_joint">
+            <command_interface name="position"/>
+            <command_interface name="velocity"/>
+            <state_interface name="position"/>
+            <state_interface name="velocity"/>
+        </joint>
     </ros2_control>
 </robot>

File: src/lotti2_control/description/urdf/Lotti_arm.xacro (robot description, xacro)
@@ -17,35 +17,33 @@
     <inertial>
       <origin
-        xyz="-0.0002249 -1.7664E-07 0.028417"
-        rpy="0 0 0" />
-      <mass
-        value="0.095547" />
-      <inertia
-        ixx="2.247E-05"
-        ixy="-3.7313E-10"
-        ixz="-2.9379E-07"
-        iyy="2.2991E-05"
-        iyz="-1.4294E-10"
-        izz="2.4917E-05" />
-    </inertial>
-    <visual>
-      <origin
-        xyz="0 0 0"
-        rpy="0 0 0" />
-      <geometry>
-        <mesh filename="package://lotti2_control/description/meshes/arm_base_link.STL" />
-      </geometry>
-      <material
-        name="">
-        <color
-          rgba="0.79216 0.81961 0.93333 1" />
-      </material>
-    </visual>
-    <collision>
-      <origin
-        xyz="0 0 0"
-        rpy="0 0 0" />
-      <geometry>
-        <mesh filename="package://lotti2_control/description/meshes/arm_base_link.STL" />
+        xyz="-0.000224896614335376 -1.76636436838296E-07 0.0284165324113623"
+        rpy="0 0 0" />
+      <mass
+        value="0.095546621133873" />
+      <inertia
+        ixx="2.24695844112508E-05"
+        ixy="-3.731322221846E-10"
+        ixz="-2.937859610971E-07"
+        iyy="2.2990565108001E-05"
+        iyz="-1.42938122280671E-10"
+        izz="2.49171374121222E-05" />
+    </inertial>
+    <visual>
+      <origin
+        xyz="0 0 0"
+        rpy="0 0 0" />
+      <geometry>
+        <mesh filename="package://lotti2_control/description/meshes/base_link.STL" />
+      </geometry>
+      <material name="">
+        <color rgba="0.792156862745098 0.819607843137255 0.933333333333333 1" />
+      </material>
+    </visual>
+    <collision>
+      <origin
+        xyz="0 0 0"
+        rpy="0 0 0" />
+      <geometry>
+        <mesh filename="package://lotti2_control/description/meshes/base_link.STL" />
       </geometry>
     </collision>
@@ -54,15 +52,15 @@
     <inertial>
       <origin
-        xyz="0.00015473 0.0066378 0.039559"
-        rpy="0 0 0" />
-      <mass
-        value="0.13887" />
-      <inertia
-        ixx="4.3388E-05"
-        ixy="2.9379E-07"
-        ixz="3.6171E-10"
-        iyy="4.8223E-05"
-        iyz="-4.4856E-06"
-        izz="4.5877E-05" />
+        xyz="-0.000148896967024248 0.0077665679059083 0.0349624287308134"
+        rpy="0 0 0" />
+      <mass
+        value="0.144567896175452" />
+      <inertia
+        ixx="4.73128961005082E-05"
+        ixy="-2.93656659450878E-07"
+        ixz="3.58678174121677E-10"
+        iyy="5.2656542855629E-05"
+        iyz="-4.39767746616673E-06"
+        izz="4.98076281467198E-05" />
     </inertial>
     <visual>
@@ -73,8 +71,6 @@
         <mesh filename="package://lotti2_control/description/meshes/arm1_link.STL" />
       </geometry>
-      <material
-        name="">
-        <color
-          rgba="0.79216 0.81961 0.93333 1" />
+      <material name="">
+        <color rgba="0.792156862745098 0.819607843137255 0.933333333333333 1" />
       </material>
     </visual>
@@ -88,8 +84,7 @@
     </collision>
   </link>
-  <joint name="arm1_joint"
-    type="revolute">
-    <origin
-      xyz="0 0 0.048"
+  <joint name="arm1_joint" type="revolute">
+    <origin
+      xyz="0 0 0.051"
       rpy="0 0 0" />
     <parent
@@ -98,8 +93,8 @@
       link="arm1_link" />
     <axis
-      xyz="0 0 -1" />
-    <limit
-      lower="-3.0"
-      upper="3.0"
+      xyz="0 0 1" />
+    <limit
+      lower="-3.2"
+      upper="3.2"
       effort="0"
       velocity="0" />
@@ -108,15 +103,15 @@
     <inertial>
       <origin
-        xyz="-0.09 0.009887 -2.6229E-15"
-        rpy="0 0 0" />
-      <mass
-        value="0.044594" />
-      <inertia
-        ixx="1.1591E-05"
-        ixy="-2.6124E-20"
-        ixz="-5.3542E-20"
-        iyy="0.00016075"
-        iyz="-9.8066E-22"
-        izz="0.00015494" />
+        xyz="-0.0900000000000001 0.00988701341491088 1.11022302462516E-16"
+        rpy="0 0 0" />
+      <mass
+        value="0.0445936683001197" />
+      <inertia
+        ixx="1.15906322136137E-05"
+        ixy="2.14234328856811E-20"
+        ixz="-8.43790123801404E-21"
+        iyy="0.000160750275623527"
+        iyz="5.85999440914565E-20"
+        izz="0.000154939805231047" />
     </inertial>
     <visual>
@@ -127,14 +122,12 @@
         <mesh filename="package://lotti2_control/description/meshes/arm2_link.STL" />
       </geometry>
-      <material
-        name="">
-        <color
-          rgba="0.79216 0.81961 0.93333 1" />
-      </material>
-    </visual>
-    <collision>
-      <origin
-        xyz="0 0 0"
-        rpy="0 0 -0.2" />
+      <material name="">
+        <color rgba="0.792156862745098 0.819607843137255 0.933333333333333 1" />
+      </material>
+    </visual>
+    <collision>
+      <origin
+        xyz="0 0 0"
+        rpy="0 0 0" />
       <geometry>
         <mesh filename="package://lotti2_control/description/meshes/arm2_link.STL" />
@@ -142,8 +135,7 @@
     </collision>
   </link>
-  <joint name="arm2_joint"
-    type="revolute">
-    <origin
-      xyz="0 0.04285 0.04755"
+  <joint name="arm2_joint" type="revolute">
+    <origin
+      xyz="0 0.04285 0.04255"
       rpy="0 0 0" />
     <parent
@@ -155,5 +147,5 @@
     <limit
       lower="-0.1"
-      upper="3.2"
+      upper="3.3"
       effort="0"
       velocity="0" />
@@ -162,15 +154,15 @@
     <inertial>
       <origin
-        xyz="0.0037748 -0.022075 0.02755"
-        rpy="0 0 0" />
-      <mass
-        value="0.23565" />
-      <inertia
-        ixx="7.7834E-05"
-        ixy="1.2652E-06"
-        ixz="-4.8745E-06"
-        iyy="7.7833E-05"
-        iyz="4.8747E-06"
-        izz="7.3141E-05" />
+        xyz="0.0034648183052334 -0.0383852430442727 0.0255502171970031"
+        rpy="0 0 0" />
+      <mass
+        value="0.245453937373138" />
+      <inertia
+        ixx="8.97316882684736E-05"
+        ixy="1.16398015613713E-06"
+        ixz="-6.81869033600654E-06"
+        iyy="8.9736154796116E-05"
+        iyz="6.8197509364556E-06"
+        izz="8.03998131737458E-05" />
     </inertial>
     <visual>
@@ -181,8 +173,6 @@
         <mesh filename="package://lotti2_control/description/meshes/arm3_link.STL" />
       </geometry>
-      <material
-        name="">
-        <color
-          rgba="0.79216 0.81961 0.93333 1" />
+      <material name="">
+        <color rgba="0.792156862745098 0.819607843137255 0.933333333333333 1" />
       </material>
     </visual>
@@ -196,9 +186,8 @@
     </collision>
   </link>
-  <joint name="arm3_joint"
-    type="revolute">
-    <origin
-      xyz="-0.18 -0.017 0"
-      rpy="0 0.0 0" />
+  <joint name="arm3_joint" type="revolute">
+    <origin
+      xyz="-0.18 0 0"
+      rpy="0 0 0" />
     <parent
       link="arm2_link" />
@@ -208,5 +197,5 @@
       xyz="0 1 0" />
     <limit
-      lower="-3.5"
+      lower="-3.3"
       upper="0.1"
       effort="0"
@@ -216,15 +205,15 @@
     <inertial>
       <origin
-        xyz="0.13759 -0.0029301 7.5985E-05"
-        rpy="0 0 0" />
-      <mass
-        value="0.14345" />
-      <inertia
-        ixx="3.2616E-05"
-        ixy="2.1538E-06"
-        ixz="8.6476E-11"
-        iyy="9.3258E-05"
-        iyz="-8.6904E-08"
-        izz="8.4066E-05" />
+        xyz="0.129288922794988 -0.00357560359269317 0.000163536166512185"
+        rpy="0 0 0" />
+      <mass
+        value="0.172732716660201" />
+      <inertia
+        ixx="4.39354110528179E-05"
+        ixy="3.80962349323384E-06"
+        ixz="-4.51308005115847E-10"
+        iyy="0.000109924099431947"
+        iyz="2.02370281934001E-10"
+        izz="0.000100955074081845" />
     </inertial>
     <visual>
@@ -235,8 +224,6 @@
         <mesh filename="package://lotti2_control/description/meshes/arm4_link.STL" />
       </geometry>
-      <material
-        name="">
-        <color
-          rgba="0.79216 0.81961 0.93333 1" />
+      <material name="">
+        <color rgba="0.792156862745098 0.819607843137255 0.933333333333333 1" />
       </material>
     </visual>
@@ -250,8 +237,7 @@
     </collision>
   </link>
-  <joint name="arm4_joint"
-    type="revolute">
-    <origin
-      xyz="0.04285 -0.02585 0.0551"
+  <joint name="arm4_joint" type="revolute">
+    <origin
+      xyz="0.04185 -0.04185 0.0511"
       rpy="0 0 0" />
     <parent
@@ -262,6 +248,6 @@
       xyz="1 0 0" />
     <limit
-      lower="-3.5"
-      upper="3.5"
+      lower="-3.3"
+      upper="3.3"
       effort="0"
       velocity="0" />
@@ -270,15 +256,15 @@
     <inertial>
       <origin
-        xyz="0.063464 0.023999 0.0010452"
-        rpy="0 0 0" />
-      <mass
-        value="0.10145" />
-      <inertia
-        ixx="2.9716E-05"
-        ixy="-6.7226E-06"
-        ixz="-1.6102E-06"
-        iyy="3.9581E-05"
-        iyz="-1.1874E-06"
-        izz="4.0743E-05" />
+        xyz="0.0572619375972157 0.0117814736268077 0.0431395601131012"
+        rpy="0 0 0" />
+      <mass
+        value="0.128456713327902" />
+      <inertia
+        ixx="8.06325333482489E-05"
+        ixy="-1.34405934586893E-05"
+        ixz="-4.06739172941076E-05"
+        iyy="0.00012665253676666"
+        iyz="-7.27945879035252E-06"
+        izz="9.1075218873226E-05" />
     </inertial>
     <visual>
@@ -289,8 +275,6 @@
         <mesh filename="package://lotti2_control/description/meshes/arm5_link.STL" />
       </geometry>
-      <material
-        name="">
-        <color
-          rgba="0.79216 0.81961 0.93333 1" />
+      <material name="">
+        <color rgba="0.792156862745098 0.819607843137255 0.933333333333333 1" />
       </material>
     </visual>
@@ -304,8 +288,7 @@
     </collision>
   </link>
-  <joint name="arm5_joint"
-    type="revolute">
-    <origin
-      xyz="0.18185 -0.0325 0"
+  <joint name="arm5_joint" type="revolute">
+    <origin
+      xyz="0.18285 -0.0247 0.0002"
       rpy="0 0 0" />
     <parent
@@ -316,6 +299,6 @@
       xyz="0 -1 0" />
     <limit
-      lower="-2.0"
-      upper="2.0"
+      lower="-3.3"
+      upper="3.3"
       effort="0"
       velocity="0" />
@@ -324,15 +307,15 @@
     <inertial>
       <origin
-        xyz="0.012243 -5.2736E-16 0"
-        rpy="0 0 0" />
-      <mass
-        value="0.016119" />
-      <inertia
-        ixx="2.0956E-06"
-        ixy="2.3665E-20"
-        ixz="3.1918E-21"
-        iyy="2.6467E-06"
-        iyz="-1.192E-14"
-        izz="2.6067E-06" />
+        xyz="0.0201016161435498 -0.00611223511695827 -0.00143428025220876"
+        rpy="0 0 0" />
+      <mass
+        value="0.0876078923434119" />
+      <inertia
+        ixx="2.73371985217545E-05"
+        ixy="4.47053107392299E-06"
+        ixz="1.79990379067894E-07"
+        iyy="2.05923742279192E-05"
+        iyz="3.38685049490894E-07"
+        izz="2.94478003276019E-05" />
     </inertial>
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
File: src/lotti2_moveit_config/config/Lotti2.ros2_control.xacro (robot description, xacro)
@@ -56,4 +56,12 @@
                 <state_interface name="velocity"/>
             </joint>
+            <joint name="arm7_joint">
+                <command_interface name="position"/>
+                <command_interface name="velocity"/>
+                <state_interface name="position">
+                  <param name="initial_value">${initial_positions['arm7_joint']}</param>
+                </state_interface>
+                <state_interface name="velocity"/>
+            </joint>
         </ros2_control>
     </xacro:macro>

Commit message: drive testing

File: src/lotti2_control/description/ros2_control/Lotti2.ros2_control.xacro (robot description, xacro)
@@ -7,5 +7,5 @@
            <!--  <param name="max_torque">0.006</param> -->
             <param name="gear_ratio">3.43</param>
-            <param name="use_hardware">1</param>
+            <param name="use_hardware">0</param>
         </hardware>
         <joint name="flipper_fr_joint">
@@ -45,5 +45,5 @@
             <param name="gear_ratio">9</param>      <!-- gearbox ratio -->
             <param name="Kt">0.198</param>          <!-- Kt value for the motor [Nm/A] -->
-            <param name="use_hardware">0</param>
+            <param name="use_hardware">1</param>
         </hardware>
         <joint name="left_chain_joint">
@@ -68,5 +68,5 @@
             <param name="gear_ratio">25.0</param>       <!-- gear ration of cycloidal gears in arm assembly -->
             <param name="resolution">16384</param>      <!-- steps per one full motor rotation-->
-            <param name="acceleration">240</param>      <!-- motor acceleration | max 255-->
+            <param name="acceleration">80</param>      <!-- motor acceleration | max 255-->
             <param name="max_motor_speed">3000</param>          <!-- motor speed in rpm | max 3000 -->
             <param name="use_hardware">0</param>        <!-- set to 1 of physical hardware is used. Set to 0 if only digital representation is used -->

File: src/lotti2_control/description/urdf/Lotti_arm.xacro (robot description, xacro)
@@ -195,8 +195,8 @@
       link="arm3_link" />
     <axis
-      xyz="0 1 0" />
-    <limit
-      lower="-3.3"
-      upper="0.1"
+      xyz="0 -1 0" />
+    <limit
+      lower="-0.1"
+      upper="3.3"
       effort="0"
       velocity="0" />
